File: hard/pcb/autopilot/main_v2.sch (EAGLE design)
At the start: 171 parts, among them IC1 24AA32ASN, IC2 INA194, IC3 LP2950Z, Q1 IRLML5203, Q3 IRLML5203, Q4 IRLML5203, T3 BC848, U2 TMP75DGK, U44 BMP085, X1 USB-SMD-NS

Commit message: Main board v2 looks finalized
Parts:
- removed R34: 30k, SparkFun:RESISTOR0805-RES
- removed R35: 1.5k, SparkFun:RESISTOR0805-RES
- removed R63: 68, SparkFun:RESISTOR0805-RES
- removed R76, R77, R79: 0, SparkFun:RESISTOR0805-RES
- added C38, C40: 0.1uF, SparkFun:CAP0805
- added DA6: AD5200, barthess:AD5200
- added VD4: BAR43, barthess:BAR43
- DA1: value (none) -> LM1117-3.3
- DD3: value (none) -> MPU9150
- JP6: value bat -> M05X2SHD; device SparkFun:JUMPER-3PTH -> barthess:M05X2SHD
- R10: value 1k -> 10k
- R31, R60: value 0 -> 68
Connections:
- removed net AN5V_3/REF: R34.2
- removed net AN_RESERVED: DD1.PC5
- removed net CAN1_RX_RESVD: DD1.PD0*
- removed net CAN1_TX_RESVD: DD1.PD1*
- removed net N$48: R34.1, R35.2, R45.1
- removed net N$76: R60.1, R63.2
- removed net N$83: DD1.VDD, R77.2, R79.2
- removed net USART2_CTS_RESVD: DD1.PD3*
- removed net USART2_RTS_RESVD: DD1.PD4*
- removed net USART2_RX_RESVD: DD1.PD6*
- removed net USART2_TX_RESVD: DD1.PD5*
- removed net VBAT: DD1.V_BAT, JP6.2
- removed net XBEE_SLEEP: JP1.9
- new net !AD_CS: DA6.!CS, DD1.PD0
- new net AD_CLK: DA6.CLK, DD1.PA3
- new net AD_SDI: DA6.SDI, DD1.PD1
- new net N$29: BAT1.+, VD4.A
- net +3.3V_A: now also DA6.A; no longer R79.1
- net 3.3V: now also C38.1, C40.1, DA6.!SHDN, DA6.VDD, DD1.VDD@1, DD1.VDD@2, DD1.VDD@3, DD1.VDD@4, DD1.VDD@5, DD1.VDD@6, DD1.V_BAT, VD4.C; no longer DD1.VDD_1, DD1.VDD_2, DD1.VDD_3, DD1.VDD_4, DD1.VDD_5
- net 5V_ENABLE: now also DD1.PA8; no longer DD1.PA8*
- net ADIS_INT: now also DD1.PE1; no longer DD1.PE1*
- net ADIS_NRST: now also DD1.PD10
- net BMP085_EOC: now also DD1.PE4; no longer DD1.PE3*
- net BOOT_1: now also DD1.BOOT_1(PB2); no longer DD1.BOOT_1(PB2)*
- net EEPROM_PWR_EN: now also DD1.PA1
- net FROM_GPS: now also DD1.PA10; no longer DD1.PA10*
- net FROM_XBEE: now also DD1.PD9; no longer DD1.PD9*
- net GND: now also C38.2, C40.2, DA6.GND, DD1.GND@1, DD1.GND@2, DD1.GND@3, DD1.GND@4, JP6.2; no longer DD1.VSS_2, DD1.VSS_3, DD1.VSS_4, DD1.VSS_5, R76.1
- net GND_A: now also DA6.B, DA6.VSS; no longer R35.1, R77.1
- net GPS_ENABLE: now also DD1.PA0
- net GPS_PPS: now also DD1.PE0; no longer DD1.PE0*
- net I2C_FAST_SCL: now also DD1.PB10; no longer DD1.PB10*
- net I2C_FAST_SDA: now also DD1.PB11; no longer DD1.PB11*
- net I2C_SLOW_SCL: now also DD1.PB6, JP6.5; no longer DD1.PB6*
- net I2C_SLOW_SDA: now also DD1.PB7, JP6.6; no longer DD1.PB7*
- net LED_B: now also DD1.PB5
- net LED_G: now also DD1.PB1
- net LED_R: now also DD1.PB0
- net MAG_INT: now also DD1.PE5; no longer DD1.PE4*
- net MPU9150_INT: now also DD1.PE3; no longer DD1.PE2*
- net N$11: now also DA6.W, R45.1; no longer BAT1.+, JP6.3
- net N$31: now also DD1.PB14; no longer DD1.PB14*
- net N$33: now also R60.1; no longer R63.1
- net N$82: no longer R76.2
- net RECEIVER_PPM: now also DD1.PB9
- net SDC_PWR_EN: now also DD1.PE15; no longer DD1.PE15*
- net SDIO_CK: now also DD1.PC12; no longer DD1.PC12*
- net SDIO_CMD: now also DD1.PD2; no longer DD1.PD2*
- net SDIO_D0: now also DD1.PC8; no longer DD1.PC8*
- net SDIO_D1: now also DD1.PC9; no longer DD1.PC9*
- net SDIO_D2: now also DD1.PC10; no longer DD1.PC10*
- net SDIO_D3: now also DD1.PC11; no longer DD1.PC11*
- net SDIO_DETECT: now also DD1.PE12; no longer DD1.PE12*
- net SONAR_PWM: now also DD1.PA2
- net SPI2_MISO_UEXT: now also JP6.7
- net SPI2_MOSI_UEXT: now also DD1.PB15, JP6.8; no longer DD1.PB15*
- net SPI2_NSS_UEXT: now also DD1.PB12, JP6.10; no longer DD1.PB12*
- net SPI2_SCK_UEXT: now also DD1.PB13, JP6.9; no longer DD1.PB13*
- net TACHOMETER: now also DD1.PB8
- net TCK: now also DD1.JTCK(PA14); no longer DD1.JTCK(PA14)*
- net TDI: now also DD1.JTDI(PA15); no longer DD1.JTDI(PA15)*
- net TDO: now also DD1.JTDO(PB3); no longer DD1.JTDO(PB3)*
- net TIM1_CH1: now also DD1.PE9; no longer DD1.PE9*
- net TIM1_CH2: now also DD1.PE11; no longer DD1.PE11*
- net TIM1_CH3: now also DD1.PE13; no longer DD1.PE13*
- net TIM1_CH4: now also DD1.PE14; no longer DD1.PE14*
- net TIM4_CH1: now also DD1.PD12; no longer DD1.PD12*
- net TIM4_CH2: now also DD1.PD13; no longer DD1.PD13*
- net TIM4_CH3: now also DD1.PD14; no longer DD1.PD14*
- net TIM4_CH4: now also DD1.PD15; no longer DD1.PD15*
- net TMP75_ALERT: now also DD1.PE6; no longer DD1.PE5*
- net TMS: now also DD1.JTMS(PA13); no longer DD1.JTMS(PA13)*
- net TO_GPS: now also DD1.PA9; no longer DD1.PA9*
- net TO_XBEE: now also DD1.PD8; no longer DD1.PD8*
- net TRST: now also DD1.NJTRST(PB4); no longer DD1.NJTRST(PB4)*
- net USART6_RX_UEXT: now also DD1.PC7, JP6.4; no longer DD1.PC7*
- net USART6_TX_UEXT: now also DD1.PC6, JP6.3; no longer DD1.PC6*
- net USB_DM: now also DD1.PA11; no longer DD1.PA11*
- net USB_DP: now also DD1.PA12; no longer DD1.PA12*
- net XBEE_CTS: now also DD1.PD11; no longer DD1.PD11*
- net XBEE_RESET: now also DD1.PD7
Other:
- note added: "an_reserved"
- note added: "usart2_cts_resvd"
- note added: "usart2_rts_resvd"
- note added: "usart2_rx_resvd"
- note added: "usart2_tx_resvd"
- note added: "xbee_sleep"
- moved on the sheet: BAT1, C1, C11, C12, C17, C2, C22, C24, C3, C4, C44, C45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

Commit message: Added board v2
Parts:
- removed C48: 0.22F/5.5v, barthess:CAP_POLIONISTOR
Connections:
- net 3.3V: no longer C48.+
- net GND: no longer C48.-
Other:
- moved on the sheet: C34
Changed lines of the file:
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@@
 <setting verticaltext="up"/>
 </settings>
-<grid distance="0.1" unitdist="inch" unit="inch" style="lines" multiple="1" display="yes" altdistance="0.01" altunitdist="inch" altunit="inch"/>
+<grid distance="0.1" unitdist="inch" unit="inch" style="lines" multiple="1" display="no" altdistance="0.01" altunitdist="inch" altunit="inch"/>
 <layers>
-<layer number="1" name="Top" color="4" fill="1" visible="no" active="no"/>
-<layer number="16" name="Bottom" color="1" fill="1" visible="no" active="no"/>
-<layer number="17" name="Pads" color="2" fill="1" visible="no" active="no"/>
-<layer number="18" name="Vias" color="2" fill="1" visible="no" active="no"/>
-<layer number="19" name="Unrouted" color="6" fill="1" visible="no" active="no"/>
-<layer number="20" name="Dimension" color="15" fill="1" visible="no" active="no"/>
-<layer number="21" name="tPlace" color="7" fill="1" visible="no" active="no"/>
-<layer number="22" name="bPlace" color="7" fill="1" visible="no" active="no"/>
-<layer number="23" name="tOrigins" color="15" fill="1" visible="no" active="no"/>
-<layer number="24" name="bOrigins" color="15" fill="1" visible="no" active="no"/>
-<layer number="25" name="tNames" color="7" fill="1" visible="no" active="no"/>
-<layer number="26" name="bNames" color="7" fill="1" visible="no" active="no"/>
-<layer number="27" name="tValues" color="7" fill="1" visible="no" active="no"/>
-<layer number="28" name="bValues" color="7" fill="1" visible="no" active="no"/>
+<layer number="1" name="Top" color="4" fill="1" visible="yes" active="no"/>
+<layer number="16" name="Bottom" color="1" fill="1" visible="yes" active="no"/>
+<layer number="17" name="Pads" color="2" fill="1" visible="yes" active="no"/>
+<layer number="18" name="Vias" color="2" fill="1" visible="yes" active="no"/>
+<layer number="19" name="Unrouted" color="6" fill="1" visible="yes" active="no"/>
+<layer number="20" name="Dimension" color="15" fill="1" visible="yes" active="no"/>
+<layer number="21" name="tPlace" color="7" fill="1" visible="yes" active="no"/>
+<layer number="22" name="bPlace" color="7" fill="1" visible="yes" active="no"/>
+<layer number="23" name="tOrigins" color="15" fill="1" visible="yes" active="no"/>
+<layer number="24" name="bOrigins" color="15" fill="1" visible="yes" active="no"/>
+<layer number="25" name="tNames" color="7" fill="1" visible="yes" active="no"/>
+<layer number="26" name="bNames" color="7" fill="1" visible="yes" active="no"/>
+<layer number="27" name="tValues" color="7" fill="1" visible="yes" active="no"/>
+<layer number="28" name="bValues" color="7" fill="1" visible="yes" active="no"/>
 <layer number="29" name="tStop" color="7" fill="3" visible="no" active="no"/>
 <layer number="30" name="bStop" color="7" fill="6" visible="no" active="no"/>
@@
 <layer number="35" name="tGlue" color="7" fill="4" visible="no" active="no"/>
 <layer number="36" name="bGlue" color="7" fill="5" visible="no" active="no"/>
-<layer number="37" name="tTest" color="7" fill="1" visible="no" active="no"/>
-<layer number="38" name="bTest" color="7" fill="1" visible="no" active="no"/>
+<layer number="37" name="tTest" color="7" fill="1" visible="yes" active="no"/>
+<layer number="38" name="bTest" color="7" fill="1" visible="yes" active="no"/>
 <layer number="39" name="tKeepout" color="4" fill="11" visible="no" active="no"/>
 <layer number="40" name="bKeepout" color="1" fill="11" visible="no" active="no"/>
@@
 <layer number="44" name="Drills" color="7" fill="1" visible="no" active="no"/>
 <layer number="45" name="Holes" color="7" fill="1" visible="no" active="no"/>
-<layer number="46" name="Milling" color="3" fill="1" visible="no" active="no"/>
-<layer number="47" name="Measures" color="7" fill="1" visible="no" active="no"/>
-<layer number="48" name="Document" color="7" fill="1" visible="no" active="no"/>
-<layer number="49" name="Reference" color="7" fill="1" visible="no" active="no"/>
-<layer number="50" name="dxf" color="7" fill="1" visible="no" active="no"/>
-<layer number="51" name="tDocu" color="14" fill="1" visible="no" active="no"/>
-<layer number="52" name="bDocu" color="7" fill="1" visible="no" active="no"/>
-<layer number="53" name="tGND_GNDA" color="7" fill="9" visible="no" active="no"/>
-<layer number="54" name="bGND_GNDA" color="1" fill="9" visible="no" active="no"/>
-<layer number="56" name="wert" color="7" fill="1" visible="no" active="no"/>
+<layer number="46" name="Milling" color="3" fill="1" visible="yes" active="no"/>
+<layer number="47" name="Measures" color="7" fill="1" visible="yes" active="no"/>
+<layer number="48" name="Document" color="7" fill="1" visible="yes" active="no"/>
+<layer number="49" name="Reference" color="7" fill="1" visible="yes" active="no"/>
+<layer number="50" name="dxf" color="7" fill="1" visible="yes" active="no"/>
+<layer number="51" name="tDocu" color="7" fill="1" visible="yes" active="no"/>
+<layer number="52" name="bDocu" color="7" fill="1" visible="yes" active="no"/>
+<layer number="53" name="tGND_GNDA" color="7" fill="9" visible="yes" active="no"/>
+<layer number="54" name="bGND_GNDA" color="1" fill="9" visible="yes" active="no"/>
+<layer number="56" name="wert" color="7" fill="1" visible="yes" active="no"/>
 <layer number="91" name="Nets" color="2" fill="1" visible="yes" active="yes"/>
 <layer number="92" name="Busses" color="1" fill="1" visible="yes" active="yes"/>
@@
 <part name="R32" library="SparkFun" deviceset="RESISTOR" device="0805-RES" value="100k"/>
 <part name="XP6" library="SparkFun" deviceset="JUMPER-3" device="PTH" value="sonar"/>
-<part name="C48" library="barthess" deviceset="CAP_POL" device="IONISTOR" value="0.22F/5.5v"/>
-<part name="GND43" library="SparkFun" deviceset="GND" device=""/>
 <part name="XP8" library="SparkFun" deviceset="JUMPER-3" device="PTH" value="PWM1"/>
 <part name="XP9" library="SparkFun" deviceset="JUMPER-3" device="PTH" value="PWM2"/>
@@
 <instance part="GND28" gate="1" x="-248.92" y="-20.32"/>
 <instance part="GND30" gate="1" x="-269.24" y="-20.32"/>
-<instance part="P+18" gate="G$1" x="-218.44" y="2.54"/>
-<instance part="GND31" gate="1" x="-218.44" y="-20.32"/>
+<instance part="P+18" gate="G$1" x="-228.6" y="2.54"/>
+<instance part="GND31" gate="1" x="-228.6" y="-20.32"/>
 <instance part="R27" gate="G$1" x="119.38" y="68.58" rot="R90"/>
 <instance part="P+16" gate="G$1" x="109.22" y="76.2"/>
@@
 <instance part="R32" gate="G$1" x="63.5" y="-76.2" rot="R270"/>
 <instance part="XP6" gate="G$1" x="-154.94" y="-170.18" rot="MR270"/>
-<instance part="C48" gate="G$1" x="-236.22" y="-10.16"/>
-<instance part="GND43" gate="1" x="-236.22" y="-20.32"/>
 <instance part="XP8" gate="G$1" x="-101.6" y="-160.02"/>
 <instance part="XP9" gate="G$1" x="-88.9" y="-160.02"/>
@@
 <instance part="JP9" gate="G$1" x="-241.3" y="-170.18" rot="R90"/>
 <instance part="C31" gate="G$1" x="-269.24" y="-10.16"/>
-<instance part="C34" gate="G$1" x="-218.44" y="-10.16"/>
+<instance part="C34" gate="G$1" x="-228.6" y="-10.16"/>
 <instance part="XP16" gate="G$1" x="-154.94" y="-160.02" rot="R90"/>
 <instance part="GND10" gate="1" x="-129.54" y="-154.94" rot="R90"/>
@@
 </segment>
 <segment>
-<wire x1="-218.44" y1="-2.54" x2="-236.22" y2="-2.54" width="0.1524" layer="91"/>
-<wire x1="-236.22" y1="-2.54" x2="-241.3" y2="-2.54" width="0.1524" layer="91"/>
-<wire x1="-218.44" y1="-7.62" x2="-218.44" y2="-2.54" width="0.1524" layer="91"/>
-<wire x1="-218.44" y1="2.54" x2="-218.44" y2="-2.54" width="0.1524" layer="91"/>
-<wire x1="-236.22" y1="-7.62" x2="-236.22" y2="-2.54" width="0.1524" layer="91"/>
-<junction x="-218.44" y="-2.54"/>
-<junction x="-218.44" y="-2.54"/>
-<junction x="-236.22" y="-2.54"/>
+<wire x1="-228.6" y1="-2.54" x2="-241.3" y2="-2.54" width="0.1524" layer="91"/>
+<wire x1="-228.6" y1="-7.62" x2="-228.6" y2="-2.54" width="0.1524" layer="91"/>
+<wire x1="-228.6" y1="2.54" x2="-228.6" y2="-2.54" width="0.1524" layer="91"/>
+<junction x="-228.6" y="-2.54"/>
+<junction x="-228.6" y="-2.54"/>
 <pinref part="P+18" gate="G$1" pin="3.3V"/>
-<pinref part="C48" gate="G$1" pin="+"/>
 <pinref part="C34" gate="G$1" pin="+"/>
 <pinref part="DA1" gate="G$1" pin="OUT"/>
@@
 </segment>
 <segment>
-<wire x1="-218.44" y1="-17.78" x2="-218.44" y2="-15.24" width="0.1524" layer="91"/>
+<wire x1="-228.6" y1="-17.78" x2="-228.6" y2="-15.24" width="0.1524" layer="91"/>
 <pinref part="GND31" gate="1" pin="GND"/>
 <pinref part="C34" gate="G$1" pin="-"/>
@@
 </segment>
 <segment>
-<wire x1="-236.22" y1="-17.78" x2="-236.22" y2="-15.24" width="0.1524" layer="91"/>
-<pinref part="GND43" gate="1" pin="GND"/>
-<pinref part="C48" gate="G$1" pin="-"/>
-</segment>
-<segment>

Commit message: Changed in PCB
Connections:
- removed net N$12: C14.+, C15.1, DA4.EN, DA4.IN, L1.2
- new net N$30: C14.+, C15.1, DA4.EN, DA4.IN, L1.2, Q1.S, R59.1
- net 6V: no longer Q1.S, R59.1
- net I2C_FAST_SCL: now also DD1.PB6; no longer DD1.PB10
- net I2C_FAST_SDA: now also DD1.PB7; no longer DD1.PB11
- net I2C_SLOW_SCL: now also DD1.PB10; no longer DD1.PB6
- net I2C_SLOW_SDA: now also DD1.PB11; no longer DD1.PB7
- net MPXV_TEMP: now also DD1.PC2; no longer DD1.PC4
- net N$54: now also DD1.PC4; no longer DD1.PC2
Other:
- moved on the sheet: C14, C15, C16, C17, C18, C22, C43, C45, DA2, DA4, IC2, L1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

Commit message: NOP
Parts:
- removed C43: 0.1uF, SparkFun:CAP0805
- removed R53: 2.2, barthess:RESISTOR1206
- removed R6: 330, SparkFun:RESISTOR0805-RES
- added C41: 10uF, SparkFun:CAP1206
- added C42: 0.1uF, SparkFun:CAP0805
- C31: value 330uF/16v -> 330uF/10v; device SparkFun:CAP_POLPTH4 -> barthess:CAP_POL7343
- C34: value 560uF/4v -> 470uF/6.3v; device rcl:CPOL-USE3.5-8 -> barthess:CAP_POL7343
- L1: device SparkFun:INDUCTOR1210 -> ferrite:EXC3BP
- ZQ1: device barthess:CRYSTALHC49UV -> crystal:CRYSTAL5X3
- ZQ2: device barthess:CRYSTALTC38H -> crystal:CRYSTAL3.2X.1.5
Connections:
- removed net N$38: C43.1, R53.1
- removed net N$8: C12.2, R6.1, ZQ1.2
- net +3.3V_A: now also C41.1, DA6.!SHDN; no longer R53.2
- net 3.3V: no longer DA6.!SHDN
- net 6V: now also C42.1
- net GND: now also C42.2
- net GND_A: now also C41.2; no longer C43.2
- net I2C_FAST_SCL: now also DD5.SCL
- net I2C_FAST_SDA: now also DD5.SDA
- net I2C_SLOW_SCL: no longer DD5.SCL
- net I2C_SLOW_SDA: no longer DD5.SDA
- net N$1: now also ZQ2.P$2; no longer ZQ2.2
- net N$6: now also ZQ2.P$1; no longer ZQ2.1
- net N$7: now also C12.2, ZQ1.P$2; no longer R6.2
- net N$9: now also ZQ1.P$1; no longer ZQ1.1
Other:
- moved on the sheet: C11, C12, C34, C51, C55, DA1

Commit message: Board v2
Connections:
- removed net N$33: R60.1, U$7.GRN
- removed net N$57: R30.1, U$7.RED
- new net N$12: R60.1, U$7.RED
- new net N$8: R30.1, U$7.GRN
- net CURRENT_SENS: now also DD1.PC2; no longer DD1.PC0
- net MPXV_TEMP: now also DD1.PC1; no longer DD1.PC2
- net N$52: now also DD1.PC3; no longer DD1.PC1
- net PRESS_DIFF: now also DD1.PC0; no longer DD1.PC3
Other:
- moved on the sheet: R30, R54, R60
Changed lines of the file:
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@@
 <instance part="R47" gate="G$1" x="345.44" y="-251.46" rot="MR90"/>
 <instance part="R48" gate="G$1" x="325.12" y="-243.84" rot="MR0"/>
-<instance part="R54" gate="G$1" x="119.38" y="-40.64"/>
+<instance part="R54" gate="G$1" x="119.38" y="-45.72"/>
 <instance part="R55" gate="G$1" x="119.38" y="-48.26"/>
 <instance part="R56" gate="G$1" x="111.76" y="-58.42" rot="R90"/>
@@
 <instance part="U$7" gate="G$1" x="198.12" y="96.52" rot="MR180"/>
 <instance part="P+23" gate="G$1" x="213.36" y="99.06" rot="MR90"/>
-<instance part="R30" gate="G$1" x="165.1" y="96.52" rot="MR0"/>
+<instance part="R30" gate="G$1" x="165.1" y="101.6" rot="MR0"/>
 <instance part="R31" gate="G$1" x="175.26" y="99.06" rot="MR0"/>
-<instance part="R60" gate="G$1" x="165.1" y="101.6" rot="MR0"/>
+<instance part="R60" gate="G$1" x="165.1" y="96.52" rot="MR0"/>
 <instance part="T3" gate="G$1" x="-302.26" y="-96.52"/>
 <instance part="R61" gate="G$1" x="-312.42" y="-96.52" rot="R180"/>
@@
 </segment>
 <segment>
-<label x="48.26" y="-45.72" size="1.27" layer="95" xref="yes"/>
-<wire x1="48.26" y1="-45.72" x2="40.64" y2="-45.72" width="0.1524" layer="91"/>
-<pinref part="DD1" gate="G$1" pin="PC3"/>
+<label x="48.26" y="-38.1" size="1.27" layer="95" xref="yes"/>
+<wire x1="48.26" y1="-38.1" x2="40.64" y2="-38.1" width="0.1524" layer="91"/>
+<pinref part="DD1" gate="G$1" pin="PC0"/>
 </segment>
 </net>
@@
 <net name="MAIN_SUPPLY" class="0">
 <segment>
-<wire x1="124.46" y1="-40.64" x2="127" y2="-40.64" width="0.1524" layer="91"/>
-<label x="127" y="-40.64" size="1.27" layer="95" xref="yes"/>
+<wire x1="124.46" y1="-45.72" x2="127" y2="-45.72" width="0.1524" layer="91"/>
+<label x="127" y="-45.72" size="1.27" layer="95" xref="yes"/>
 <pinref part="R54" gate="G$1" pin="2"/>
 </segment>
@@
 <net name="N$52" class="0">
 <segment>
-<wire x1="114.3" y1="-40.64" x2="111.76" y2="-40.64" width="0.1524" layer="91"/>
-<wire x1="111.76" y1="-53.34" x2="111.76" y2="-40.64" width="0.1524" layer="91"/>
-<wire x1="40.64" y1="-40.64" x2="101.6" y2="-40.64" width="0.1524" layer="91"/>
-<junction x="111.76" y="-40.64"/>
+<wire x1="114.3" y1="-45.72" x2="111.76" y2="-45.72" width="0.1524" layer="91"/>
+<wire x1="111.76" y1="-53.34" x2="111.76" y2="-45.72" width="0.1524" layer="91"/>
+<junction x="111.76" y="-45.72"/>
 <pinref part="R54" gate="G$1" pin="1"/>
 <pinref part="R56" gate="G$1" pin="2"/>
 <pinref part="VD2" gate="G$1" pin="C"/>
-<wire x1="101.6" y1="-40.64" x2="106.68" y2="-40.64" width="0.1524" layer="91"/>
-<wire x1="106.68" y1="-40.64" x2="111.76" y2="-40.64" width="0.1524" layer="91"/>
-<wire x1="101.6" y1="-55.88" x2="101.6" y2="-40.64" width="0.1524" layer="91"/>
-<junction x="101.6" y="-40.64"/>
-<pinref part="DD1" gate="G$1" pin="PC1"/>
+<wire x1="101.6" y1="-45.72" x2="106.68" y2="-45.72" width="0.1524" layer="91"/>
+<wire x1="106.68" y1="-45.72" x2="111.76" y2="-45.72" width="0.1524" layer="91"/>
+<wire x1="101.6" y1="-55.88" x2="101.6" y2="-45.72" width="0.1524" layer="91"/>
 <pinref part="C37" gate="G$1" pin="2"/>
-<wire x1="106.68" y1="-53.34" x2="106.68" y2="-40.64" width="0.1524" layer="91"/>
-<junction x="106.68" y="-40.64"/>
+<wire x1="106.68" y1="-53.34" x2="106.68" y2="-45.72" width="0.1524" layer="91"/>
+<junction x="106.68" y="-45.72"/>
+<pinref part="DD1" gate="G$1" pin="PC3"/>
+<wire x1="101.6" y1="-45.72" x2="40.64" y2="-45.72" width="0.1524" layer="91"/>
+<junction x="101.6" y="-45.72"/>
 </segment>
 </net>
@@
 </segment>
 </net>
-<net name="N$57" class="0">
-<segment>
-<wire x1="187.96" y1="96.52" x2="170.18" y2="96.52" width="0.1524" layer="91"/>
-<pinref part="U$7" gate="G$1" pin="RED"/>
-<pinref part="R30" gate="G$1" pin="1"/>
-</segment>
-</net>
 <net name="LED_G" class="0">
 <segment>
-<wire x1="160.02" y1="101.6" x2="157.48" y2="101.6" width="0.1524" layer="91"/>
-<label x="157.48" y="101.6" size="1.27" layer="95" rot="MR0" xref="yes"/>
+<wire x1="160.02" y1="96.52" x2="157.48" y2="96.52" width="0.1524" layer="91"/>
+<label x="157.48" y="96.52" size="1.27" layer="95" rot="MR0" xref="yes"/>
 <pinref part="R60" gate="G$1" pin="2"/>
 </segment>
@@
 <net name="LED_R" class="0">
 <segment>
-<wire x1="160.02" y1="96.52" x2="157.48" y2="96.52" width="0.1524" layer="91"/>
-<label x="157.48" y="96.52" size="1.27" layer="95" rot="MR0" xref="yes"/>
+<wire x1="160.02" y1="101.6" x2="157.48" y2="101.6" width="0.1524" layer="91"/>
+<label x="157.48" y="101.6" size="1.27" layer="95" rot="MR0" xref="yes"/>
 <pinref part="R30" gate="G$1" pin="2"/>
 </segment>
@@
 </segment>
 <segment>
-<wire x1="40.64" y1="-38.1" x2="48.26" y2="-38.1" width="0.1524" layer="91"/>
-<label x="48.26" y="-38.1" size="1.27" layer="95" xref="yes"/>
-<pinref part="DD1" gate="G$1" pin="PC0"/>
+<label x="48.26" y="-43.18" size="1.27" layer="95" xref="yes"/>
+<pinref part="DD1" gate="G$1" pin="PC2"/>
+<wire x1="48.26" y1="-43.18" x2="40.64" y2="-43.18" width="0.1524" layer="91"/>
 </segment>
 </net>
@@
 </segment>
 </net>
-<net name="N$33" class="0">
-<segment>
-<pinref part="U$7" gate="G$1" pin="GRN"/>
-<pinref part="R60" gate="G$1" pin="1"/>
-<wire x1="187.96" y1="101.6" x2="170.18" y2="101.6" width="0.1524" layer="91"/>
-</segment>
-</net>
 <net name="N$78" class="0">
 <segment>
@@
 </segment>
 <segment>
-<label x="48.26" y="-43.18" size="1.27" layer="95" xref="yes"/>
-<wire x1="48.26" y1="-43.18" x2="40.64" y2="-43.18" width="0.1524" layer="91"/>
-<pinref part="DD1" gate="G$1" pin="PC2"/>
+<pinref part="DD1" gate="G$1" pin="PC1"/>
+<wire x1="48.26" y1="-40.64" x2="40.64" y2="-40.64" width="0.1524" layer="91"/>
+<label x="48.26" y="-40.64" size="1.27" layer="95" xref="yes"/>
 </segment>
 </net>
@@
 </segment>
 </net>
+<net name="N$8" class="0">
+<segment>
+<pinref part="R30" gate="G$1" pin="1"/>
+<pinref part="U$7" gate="G$1" pin="GRN"/>
+<wire x1="170.18" y1="101.6" x2="187.96" y2="101.6" width="0.1524" layer="91"/>
+</segment>
+</net>
+<net name="N$12" class="0">
+<segment>
+<pinref part="R60" gate="G$1" pin="1"/>
+<pinref part="U$7" gate="G$1" pin="RED"/>
+<wire x1="170.18" y1="96.52" x2="187.96" y2="96.52" width="0.1524" layer="91"/>
+</segment>
+</net>
