File: hard/pcb/autopilot/main_v2.sch (EAGLE design)
At the start: 167 parts, among them IC1 24AA32ASN, IC2 INA194, IC3 LP2950Z, Q1 IRLML5203, Q3 IRLML5203, Q4 IRLML5203, T3 BC848, U2 TMP75DGK, U44 BMP085, X1 USB-SMD-NS

Commit message: board v2 nop
Connections:
- new net N$33: C40.1, DD1.V_BAT, VD4.C
- net 3.3V: no longer C40.1, DD1.V_BAT, VD4.C
Changed lines of the file:
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@@
 <part name="VD4" library="barthess" deviceset="BAR43" device=""/>
 <part name="C40" library="SparkFun" deviceset="CAP" device="0805" value="0.1uF"/>
-<part name="P+21" library="SparkFun" deviceset="3.3V" device=""/>
 <part name="JP6" library="barthess" deviceset="M05X2" device="SHD"/>
 <part name="P+22" library="SparkFun" deviceset="3.3V" device=""/>
@@
 <instance part="VD4" gate="1" x="-73.66" y="68.58"/>
 <instance part="C40" gate="G$1" x="-53.34" y="63.5" rot="MR0"/>
-<instance part="P+21" gate="G$1" x="-53.34" y="71.12"/>
 <instance part="JP6" gate="G$1" x="198.12" y="195.58"/>
 <instance part="P+22" gate="G$1" x="185.42" y="200.66"/>
@@
 <pinref part="P+8" gate="G$1" pin="3.3V"/>
 <wire x1="289.56" y1="-208.28" x2="289.56" y2="-213.36" width="0.1524" layer="91"/>
-</segment>
-<segment>
-<pinref part="DD1" gate="G$1" pin="V_BAT"/>
-<wire x1="-33.02" y1="68.58" x2="-53.34" y2="68.58" width="0.1524" layer="91"/>
-<pinref part="VD4" gate="1" pin="C"/>
-<pinref part="C40" gate="G$1" pin="1"/>
-<wire x1="-53.34" y1="68.58" x2="-71.12" y2="68.58" width="0.1524" layer="91"/>
-<junction x="-53.34" y="68.58"/>
-<pinref part="P+21" gate="G$1" pin="3.3V"/>
-<wire x1="-53.34" y1="68.58" x2="-53.34" y2="71.12" width="0.1524" layer="91"/>
 </segment>
 <segment>
@@
 </segment>
 </net>
+<net name="N$33" class="0">
+<segment>
+<pinref part="DD1" gate="G$1" pin="V_BAT"/>
+<wire x1="-33.02" y1="68.58" x2="-53.34" y2="68.58" width="0.1524" layer="91"/>
+<pinref part="VD4" gate="1" pin="C"/>
+<pinref part="C40" gate="G$1" pin="1"/>
+<wire x1="-53.34" y1="68.58" x2="-71.12" y2="68.58" width="0.1524" layer="91"/>
+<junction x="-53.34" y="68.58"/>
+</segment>
+</net>

Commit message: board v2. nop
Parts:
- removed C49: 2.2uF, rcl:C-EUC1206
- added C43: 2.2uF, SparkFun:CAP0805
Connections:
- net GND_A: now also C43.2; no longer C49.1
- net N$47: now also C43.1; no longer C49.2
Changed lines of the file:
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@@
 <class number="0" name="default" width="0" drill="0">
+</class>
+<class number="1" name="+5V_A" width="0.4" drill="0.5">
+</class>
+<class number="2" name="+3.3V_A" width="0.4" drill="0.5">
+</class>
+<class number="3" name="GND_A" width="0.4" drill="0.5">
 </class>
 </classes>
@@
 <part name="R33" library="SparkFun" deviceset="RESISTOR" device="0805-RES" value="100k"/>
 <part name="R45" library="SparkFun" deviceset="RESISTOR" device="0805-RES" value="10k"/>
-<part name="C49" library="rcl" deviceset="C-EU" device="C1206" value="2.2uF"/>
 <part name="C50" library="SparkFun" deviceset="CAP" device="0805" value="0.1uF"/>
 <part name="DA3" library="barthess" deviceset="MPXV5010DP" device=""/>
@@
 <part name="C42" library="SparkFun" deviceset="CAP" device="0805" value="0.1uF"/>
 <part name="GND29" library="SparkFun" deviceset="GND" device=""/>
+<part name="C43" library="SparkFun" deviceset="CAP" device="0805" value="2.2uF"/>
 </parts>
 <sheets>
@@
 <instance part="R33" gate="G$1" x="350.52" y="-215.9"/>
 <instance part="R45" gate="G$1" x="340.36" y="-215.9" rot="MR180"/>
-<instance part="C49" gate="G$1" x="332.74" y="-254" rot="R180"/>
 <instance part="C50" gate="G$1" x="284.48" y="-246.38"/>
 <instance part="DA3" gate="G$1" x="304.8" y="-243.84" smashed="yes">
@@
 <instance part="C42" gate="G$1" x="-256.54" y="-12.7"/>
 <instance part="GND29" gate="1" x="-256.54" y="-20.32"/>
+<instance part="C43" gate="G$1" x="332.74" y="-254"/>
 </instances>
 <busses>
@@
 </segment>
 </net>
-<net name="+3.3V_A" class="0">
+<net name="+3.3V_A" class="2">
 <segment>
 <wire x1="345.44" y1="-109.22" x2="345.44" y2="-119.38" width="0.1524" layer="91"/>
@@
 <pinref part="R48" gate="G$1" pin="1"/>
 <pinref part="R47" gate="G$1" pin="2"/>
-<pinref part="C49" gate="G$1" pin="2"/>
 <wire x1="332.74" y1="-248.92" x2="332.74" y2="-243.84" width="0.1524" layer="91"/>
 <junction x="332.74" y="-243.84"/>
@@
 <wire x1="345.44" y1="-243.84" x2="345.44" y2="-236.22" width="0.1524" layer="91"/>
 <wire x1="345.44" y1="-236.22" x2="350.52" y2="-236.22" width="0.1524" layer="91"/>
+<pinref part="C43" gate="G$1" pin="1"/>
 </segment>
 </net>
@@
 </segment>
 </net>
-<net name="GND_A" class="0">
+<net name="GND_A" class="3">
 <segment>
 <label x="-38.1" y="58.42" size="1.27" layer="95" rot="R180" xref="yes"/>
@@
 <wire x1="332.74" y1="-256.54" x2="332.74" y2="-259.08" width="0.1524" layer="91"/>
 <label x="332.74" y="-259.08" size="1.27" layer="95" rot="R270" xref="yes"/>
-<pinref part="C49" gate="G$1" pin="1"/>
+<pinref part="C43" gate="G$1" pin="2"/>
 </segment>
 <segment>
@@
 </segment>
 </net>
-<net name="+5V_A" class="0">
+<net name="+5V_A" class="1">
 <segment>
 <wire x1="-218.44" y1="-99.06" x2="-228.6" y2="-99.06" width="0.1524" layer="91"/>

Commit message: board v2 nop
Parts:
- removed R9: 0, SparkFun:RESISTOR0805-RES
- added R6: 0, barthess:RESISTOR1206
Connections:
- net GND: now also R6.2; no longer R9.1
- net GND_A: now also R6.1; no longer R9.2
Changed lines of the file:
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@@
 <part name="C14" library="SparkFun" deviceset="CAP_POL" device="1206-KIT" value="10uF/16v"/>
 <part name="C15" library="SparkFun" deviceset="CAP" device="0805" value="0.1uF"/>
-<part name="R9" library="SparkFun" deviceset="RESISTOR" device="0805-RES" value="0"/>
 <part name="L1" library="ferrite" deviceset="EXC3BP" device="" value="1uH"/>
 <part name="GND13" library="SparkFun" deviceset="GND" device=""/>
@@
 <part name="GND29" library="SparkFun" deviceset="GND" device=""/>
 <part name="C43" library="SparkFun" deviceset="CAP" device="0805" value="2.2uF"/>
+<part name="R6" library="barthess" deviceset="RESISTOR" device="1206" value="0"/>
 </parts>
 <sheets>
@@
 <instance part="C14" gate="G$1" x="-287.02" y="-60.96"/>
 <instance part="C15" gate="G$1" x="-271.78" y="-63.5"/>
-<instance part="R9" gate="G$1" x="-195.58" y="-91.44" rot="R180"/>
 <instance part="L1" gate="G$1" x="-302.26" y="-55.88"/>
 <instance part="GND13" gate="1" x="-96.52" y="60.96" rot="R270"/>
@@
 <instance part="GND29" gate="1" x="-256.54" y="-20.32"/>
 <instance part="C43" gate="G$1" x="332.74" y="-254"/>
+<instance part="R6" gate="G$1" x="-195.58" y="-91.44"/>
 </instances>
 <busses>
@@
 </segment>
 <segment>
-<pinref part="R9" gate="G$1" pin="1"/>
 <pinref part="GND11" gate="1" pin="GND"/>
 <wire x1="-190.5" y1="-91.44" x2="-187.96" y2="-91.44" width="0.1524" layer="91"/>
+<pinref part="R6" gate="G$1" pin="2"/>
 </segment>
 <segment>
@@
 <wire x1="-203.2" y1="-114.3" x2="-203.2" y2="-91.44" width="0.1524" layer="91"/>
 <junction x="-203.2" y="-73.66"/>
-<pinref part="R9" gate="G$1" pin="2"/>
 <wire x1="-203.2" y1="-91.44" x2="-203.2" y2="-73.66" width="0.1524" layer="91"/>
 <wire x1="-200.66" y1="-91.44" x2="-203.2" y2="-91.44" width="0.1524" layer="91"/>
@@
 <wire x1="-248.92" y1="-111.76" x2="-248.92" y2="-114.3" width="0.1524" layer="91"/>
 <junction x="-248.92" y="-114.3"/>
-</segment>
-<segment>
+<pinref part="R6" gate="G$1" pin="1"/>
+</segment>
+<segment>
