File: hard/pcb/autopilot/main_v2.brd (EAGLE design)
At the start: 100 x 65 mm, 168 parts, among them IC1 24AA32ASN, IC2 INA194, IC3 LP2950Z, Q1 IRLML5203, Q3 IRLML5203, Q4 IRLML5203, T3 BC848, U2 TMP75DGK, U44 BMP085, X1 USB-SMD-NS

Commit message: cosmetical improvements
Parts:
- moved R42 9.00 mm to (22.0, 55.5)
- moved XP12 9.00 mm to (21.0, 58.0)
- moved R44 6.00 mm to (28.0, 55.5)
- moved XP14 6.00 mm to (27.0, 58.0)
- moved R46 3.00 mm to (31.0, 55.5)
- moved XP15 3.00 mm to (30.0, 58.0)
Routing:
- net TIM4_CH1: track 18.4 -> 27.4 mm
- net TIM4_CH3: track 28.7 -> 22.7 mm
- net TIM4_CH4: track 22.9 -> 19.5 mm
Other:
- board text added: "+"
- board text added: "-"
- board text added: "Boot_0"
- board text added: "Boot_1"
- board text added: "Current"
- board text added: "GPS"
- board text added: "PWM"
- board text added: "PWM1-1"
- board text added: "PWM1-2"
- board text added: "PWM1-3"
- board text added: "PWM1-4"
- board text added: "PWM4-1"
- board text added: "PWM4-2"
- board text added: "PWM4-3"
- board text added: "PWM4-4"
- board text added: "Power"
- board text added: "RC-PPM"
- board text added: "Sonar"
- board text added: "Tacho"
- board text added: "Xbee"

Commit message: Main board. Final cut
Parts:
- R6, R64: device barthess:R1206 -> barthess:1206
- XP1: device barthess:2X10-PSEUDOSMD -> barthess:PLD_2X10_PSEUDOSMD
- XP18: device barthess:1X02 -> barthess:PLD_1X02
- moved U$2 1.50 mm to (60.5, 11.6)
Other:
- board text added: "RC"
- board text removed: "PWM"
- board text removed: "RC-PPM"

Commit message: Nop
Parts:
- JP3, JP7, JP8, JP9: value STAND-OFFTIGHT -> STAND-OFF; device SparkFun:STAND-OFF-TIGHT -> barthess:STAND-OFF
- JP4, JP5, XP10, XP11, XP12, XP13, XP14, XP15, XP16, XP17, XP2, XP6, XP8, XP9: device SparkFun:1X03 -> barthess:PLD_1X03
Changed lines of the file:
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@@
 <layer number="37" name="tTest" color="7" fill="1" visible="no" active="yes"/>
 <layer number="38" name="bTest" color="7" fill="1" visible="no" active="yes"/>
-<layer number="39" name="tKeepout" color="4" fill="11" visible="no" active="yes"/>
-<layer number="40" name="bKeepout" color="1" fill="11" visible="no" active="yes"/>
-<layer number="41" name="tRestrict" color="4" fill="10" visible="no" active="yes"/>
-<layer number="42" name="bRestrict" color="1" fill="10" visible="no" active="yes"/>
+<layer number="39" name="tKeepout" color="4" fill="11" visible="yes" active="yes"/>
+<layer number="40" name="bKeepout" color="1" fill="11" visible="yes" active="yes"/>
+<layer number="41" name="tRestrict" color="4" fill="10" visible="yes" active="yes"/>
+<layer number="42" name="bRestrict" color="1" fill="10" visible="yes" active="yes"/>
 <layer number="43" name="vRestrict" color="2" fill="10" visible="no" active="yes"/>
 <layer number="44" name="Drills" color="7" fill="1" visible="yes" active="yes"/>
@@
 <element name="R2" library="SparkFun" package="0805" value="10k" x="31.8" y="21.1"/>
 <element name="R3" library="SparkFun" package="0805" value="10k" x="31.8" y="29.1"/>
-<element name="JP4" library="SparkFun" package="1X03" value="boot_0" x="25.8" y="26.6"/>
-<element name="JP5" library="SparkFun" package="1X03" value="boot_1" x="25.8" y="23.6"/>
+<element name="JP4" library="barthess" package="PLD_1X03" value="boot_0" x="25.8" y="26.6"/>
+<element name="JP5" library="barthess" package="PLD_1X03" value="boot_1" x="25.8" y="23.6"/>
 <element name="R5" library="SparkFun" package="0805" value="100" x="28.8" y="29.1" rot="R180"/>
 <element name="R4" library="SparkFun" package="0805" value="100" x="28.8" y="21.1" rot="R180"/>
@@
 <attribute name="PARTNO" value="?" x="95.6" y="41.7" size="1.778" layer="28" rot="MR90" display="off"/>
 </element>
-<element name="XP2" library="SparkFun" package="1X03" value="RECEIVER" x="98.16" y="38.34" rot="R90"/>
+<element name="XP2" library="barthess" package="PLD_1X03" value="RECEIVER" x="98.16" y="38.34" rot="R90"/>
 <element name="R29" library="SparkFun" package="0805" value="1k" x="95.5" y="38" rot="MR0"/>
 <element name="R32" library="SparkFun" package="0805" value="100k" x="68.43" y="33.65" rot="MR225"/>
-<element name="XP6" library="SparkFun" package="1X03" value="sonar" x="47.8" y="7.4" rot="R270"/>
-<element name="XP8" library="SparkFun" package="1X03" value="PWM1" x="9" y="58" rot="R90"/>
-<element name="XP9" library="SparkFun" package="1X03" value="PWM2" x="12" y="58" rot="R90"/>
-<element name="XP10" library="SparkFun" package="1X03" value="PWM3" x="15" y="58" rot="R90"/>
-<element name="XP11" library="SparkFun" package="1X03" value="PWM4" x="18" y="58" rot="R90"/>
-<element name="XP12" library="SparkFun" package="1X03" value="PWM5" x="21" y="58" rot="R90"/>
-<element name="XP13" library="SparkFun" package="1X03" value="PWM6" x="24" y="58" rot="R90"/>
-<element name="XP14" library="SparkFun" package="1X03" value="PWM7" x="27" y="58" rot="R90"/>
-<element name="XP15" library="SparkFun" package="1X03" value="PWM8" x="30" y="58" rot="R90"/>
+<element name="XP6" library="barthess" package="PLD_1X03" value="sonar" x="47.8" y="7.4" rot="R270"/>
+<element name="XP8" library="barthess" package="PLD_1X03" value="PWM1" x="9" y="58" rot="R90"/>
+<element name="XP9" library="barthess" package="PLD_1X03" value="PWM2" x="12" y="58" rot="R90"/>
+<element name="XP10" library="barthess" package="PLD_1X03" value="PWM3" x="15" y="58" rot="R90"/>
+<element name="XP11" library="barthess" package="PLD_1X03" value="PWM4" x="18" y="58" rot="R90"/>
+<element name="XP12" library="barthess" package="PLD_1X03" value="PWM5" x="21" y="58" rot="R90"/>
+<element name="XP13" library="barthess" package="PLD_1X03" value="PWM6" x="24" y="58" rot="R90"/>
+<element name="XP14" library="barthess" package="PLD_1X03" value="PWM7" x="27" y="58" rot="R90"/>
+<element name="XP15" library="barthess" package="PLD_1X03" value="PWM8" x="30" y="58" rot="R90"/>
 <element name="R33" library="SparkFun" package="0805" value="100k" x="83" y="11" rot="MR270"/>
 <element name="R45" library="SparkFun" package="0805" value="10k" x="87" y="9.5" rot="MR0"/>
@@
 <element name="S2" library="barthess" package="BUTTON_6X3.5" value="RESET" x="1.79" y="45.98"/>
 <element name="C24" library="SparkFun" package="0805" value="0.1uF" x="88.75" y="14.75" rot="MR0"/>
-<element name="XP17" library="SparkFun" package="1X03" value="power" x="33" y="58" rot="R90"/>
+<element name="XP17" library="barthess" package="PLD_1X03" value="power" x="33" y="58" rot="R90"/>
 <element name="R36" library="SparkFun" package="0805" value="47" x="72.5" y="5.75" rot="MR90"/>
 <element name="R51" library="SparkFun" package="0805" value="47" x="75.25" y="5.75" rot="MR90"/>
@@
 <element name="C45" library="SparkFun" package="1206" value="10uF" x="74" y="8.75" rot="MR180"/>
 <element name="XP18" library="barthess" package="PLD_1X02" value="current_sens" x="72.75" y="2.75"/>
-<element name="JP3" library="SparkFun" package="STAND-OFF-TIGHT" value="STAND-OFFTIGHT" x="4" y="61"/>
-<element name="JP7" library="SparkFun" package="STAND-OFF-TIGHT" value="STAND-OFFTIGHT" x="96" y="61"/>
-<element name="JP8" library="SparkFun" package="STAND-OFF-TIGHT" value="STAND-OFFTIGHT" x="4" y="4"/>
-<element name="JP9" library="SparkFun" package="STAND-OFF-TIGHT" value="STAND-OFFTIGHT" x="96" y="4"/>
+<element name="JP3" library="barthess" package="STAND-OFF" value="STAND-OFF" x="4" y="61"/>
+<element name="JP7" library="barthess" package="STAND-OFF" value="STAND-OFF" x="96" y="61"/>
+<element name="JP8" library="barthess" package="STAND-OFF" value="STAND-OFF" x="4" y="4"/>
+<element name="JP9" library="barthess" package="STAND-OFF" value="STAND-OFF" x="96" y="4"/>
 <element name="C31" library="barthess" package="EIA7343" value="330uF/10v" x="63.01" y="58.85" rot="MR90"/>
 <element name="C34" library="barthess" package="EIA7343" value="470uF/6.3v" x="84.24" y="51.41" rot="MR90"/>
-<element name="XP16" library="SparkFun" package="1X03" value="tacho" x="44.8" y="7.4" rot="R270"/>
+<element name="XP16" library="barthess" package="PLD_1X03" value="tacho" x="44.8" y="7.4" rot="R270"/>
 <element name="R75" library="SparkFun" package="0805" value="1k" x="79.8" y="32.2" rot="MR180"/>
 <element name="R64" library="barthess" package="1206" value="0" x="38.5" y="63"/>
