File: hard/pcb/kalman/main_v2.brd (EAGLE design)
At the start: 100 x 65 mm, 39 parts, among them X1 USB-SMD-NS

Commit message: PCB routed
Parts:
- removed JP2: 2X5, barthess:PLD_2X05_PSEUDOSMD
- removed JP3, JP9: STAND-OFF, barthess:STAND-OFF
- removed R12, R13: 33, SparkFun:0805
- removed U$2: (no value), barthess:LOGO_CHIBIOS_SILK
- added JP1, JP10, JP11, JP12, JP14, JP15, JP16, JP17, JP18, JP19, JP20, JP22, JP4, JP5, JP6: M01OFFSET, SparkFun-Connectors:1X01_OFFSET
- added R10, R11, R14, R15, R16, R17, R18, R19, R2, R20, R21, R22, R23, R24, R25, R26, R27, R28, R29, R3, R31, R32, R33, R34, R35, R36, R37, R39, R4, R40, R41, R42, R43, R5, R6, R8, R9: 1k, SparkFun:0805
- added VD1, VD2: (no value), led:LED-1206
- U$4: device barthess:TQFP176 -> barthess:TQFP176(1.5X0.25)
- ZQ1: device crystal:86SMX -> crystal:CTS406
- moved C26 149.2 mm to (69.0, 43.5), flipped to the bottom
- moved C25 135.7 mm to (68.0, 27.0), flipped to the bottom, turned to 270 degrees
- moved C18 131.1 mm to (62.0, 51.5), flipped to the bottom, turned to 270 degrees
- moved C24 124.7 mm to (62.5, 19.5), flipped to the bottom
- moved C15 121.9 mm to (68.5, 34.3), flipped to the bottom, turned to 270 degrees
- moved C17 118.8 mm to (50.0, 51.0), flipped to the bottom, turned to 180 degrees
- moved C22 117.7 mm to (56.7, 19.5), flipped to the bottom
- moved C8 117.4 mm to (69.5, 40.2), flipped to the bottom, turned to 270 degrees
- moved C9 111.9 mm to (55.5, 51.0), flipped to the bottom, turned to 180 degrees
- moved C16 111.2 mm to (43.0, 51.5), flipped to the bottom, turned to 180 degrees
- moved C20 108.0 mm to (37.5, 37.0), flipped to the bottom, turned to 90 degrees
- moved C21 103.3 mm to (38.5, 24.5), flipped to the bottom, turned to 90 degrees
- moved C19 101.3 mm to (37.7, 30.3), flipped to the bottom, turned to 90 degrees
- moved C14 97.2 mm to (36.2, 45.2), flipped to the bottom, turned to 180 degrees
- moved C10 96.1 mm to (49.8, 18.0), flipped to the bottom
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Connections:
- net RESET renamed NRST
- removed net FROM_GPS: JP2.2
- removed net GPS_ENABLE: JP2.7
- removed net GPS_PPS: JP2.4
- removed net PDR_ON: U$4.171
- removed net TCK: XP1.9
- removed net TDI: XP1.5
- removed net TDO: XP1.13
- removed net TMS: XP1.7
- removed net TO_GPS: JP2.3
- removed net TRST: XP1.3
- new net !CE: R43.1, U$4.151
- new net !LB: R39.1, U$4.169
- new net !OE: R41.1, U$4.146
- new net !UB: R40.1, U$4.170
- new net !WE: R42.1, U$4.147
- new net A0: R21.2, U$4.16
- new net A1: R22.2, U$4.17
- new net A10: R32.2, U$4.66
- new net A11: R33.2, U$4.67
- new net A12: R34.2, U$4.106
- new net A13: R35.2, U$4.107
- new net A14: R36.2, U$4.108
- new net A15: R37.2, U$4.109
- new net A2: R23.2, U$4.18
- new net A3: R24.2, U$4.19
- new net A4: R25.2, U$4.20
- new net A5: R26.2, U$4.21
- new net A6: R27.2, U$4.60
- new net A7: R28.2, U$4.63
- new net A8: R29.2, U$4.64
- new net A9: R31.2, U$4.65
- new net D0: R2.2, U$4.104
- new net D1: R3.2, U$4.105
- new net D10: R15.2, U$4.76
- new net D11: R16.2, U$4.77
- new net D12: R17.2, U$4.78
- new net D13: R18.2, U$4.96
- new net D14: R19.2, U$4.97
- new net D15: R20.2, U$4.98
- new net D2: R4.2, U$4.142
- new net D3: R5.2, U$4.143
- new net D4: R6.2, U$4.68
- new net D5: R8.2, U$4.69
- new net D6: R9.2, U$4.70
- new net D7: R10.2, U$4.73
- new net D8: R11.2, U$4.74
- new net D9: R14.2, U$4.75
- new net ISR_KALMAN: JP11.1, U$4.133
- new net ISR_UART: JP12.1, U$4.134
- new net JTCK: U$4.137, XP1.9
- new net JTDI: U$4.138, XP1.5
- new net JTDO: U$4.161, XP1.13
- new net JTMS: U$4.124, XP1.7
- new net JTRST: U$4.162, XP1.3
- new net N$11: R9.1, U$3.36
- new net N$14: R10.1, U$3.34
- new net N$15: R11.1, U$3.32
- new net N$16: R14.1, U$3.30
- new net N$17: R15.1, U$3.28
- new net N$18: R16.1, U$3.26
- new net N$19: R17.1, U$3.24
- new net N$20: R20.1, U$3.14
- new net N$23: R2.1, U$3.12
- new net N$24: R3.1, U$3.10
- new net N$25: R23.1, U$3.60
- new net N$26: R24.1, U$3.58
- new net N$27: R25.1, U$3.56
- new net N$28: R26.1, U$3.54
- new net N$29: R27.1, U$3.52
- new net N$3: JP1.1, R43.2
- new net N$30: R28.1, U$3.50
- new net N$32: R29.1, U$3.48
- new net N$33: R31.1, U$3.46
- new net N$34: R32.1, U$3.44
- new net N$35: R33.1, U$3.42
- new net N$36: R34.1, U$3.8
- new net N$37: R35.1, U$3.6
- new net N$38: R36.1, U$3.4
- new net N$39: R37.1, U$3.2
- new net N$4: R5.1, U$3.22
- new net N$42: JP4.1, R42.2
- new net N$43: JP5.1, R41.2
- new net N$44: JP6.1, R40.2
- new net N$45: JP10.1, R39.2
- new net N$5: R4.1, U$3.20
- new net N$6: R18.1, U$3.18
- new net N$7: R19.1, U$3.16
- new net N$8: R6.1, U$3.40
- new net N$9: R8.1, U$3.38
- net 3.3V: now also JP22.1, U$4.171; no longer JP2.1
- net GND: now also JP14.1, JP15.1, JP16.1, JP17.1, JP18.1, JP19.1, JP20.1, U$3.1, U$3.11, U$3.13, U$3.15, U$3.17, U$3.19, U$3.21, U$3.23, U$3.25, U$3.27, U$3.29, U$3.3, U$3.31, U$3.33, U$3.35, U$3.37, U$3.39, U$3.41, U$3.43, U$3.45, U$3.47, U$3.49, U$3.5, U$3.51, U$3.53, U$3.55, U$3.57, U$3.59, U$3.61, U$3.63, U$3.7, U$3.9, VD1.C, VD2.C; no longer JP2.10
- net LED_G: now also U$4.2
- net LED_R: now also U$4.1
- net N$10: now also R21.1, U$3.64; no longer R12.1, X1.D-
- net N$12: now also VD1.A
- net N$13: now also R22.1, U$3.62; no longer R13.1, X1.D+
- net N$21: now also ZQ1.3; no longer ZQ1.4
- net N$31: now also VD2.A
- net USB_DM: now also X1.D-; no longer R12.2
- net USB_DP: now also X1.D+; no longer R13.2
- net USB_PRESENT: now also U$4.121
Routing:
- net 3.3V: track 0.00 -> 202.1 mm, vias 0 -> 3
- net NRST: track 8.13 -> 77.2 mm, vias 0 -> 2
- net !UB: track 0.00 -> 68.1 mm
- net JTRST: track 0.00 -> 67.7 mm, vias 0 -> 2
- net !LB: track 0.00 -> 65.1 mm
- net !CE: track 0.00 -> 55.1 mm
- net D2: track 0.00 -> 49.9 mm
- net A15: track 0.00 -> 49.5 mm
- net D3: track 0.00 -> 49.0 mm
- net GND: track 0.00 -> 48.1 mm, vias 24 -> 7
- net !WE: track 0.00 -> 47.9 mm
- net A14: track 0.00 -> 46.8 mm
- net A0: track 0.00 -> 45.6 mm
- net A1: track 0.00 -> 45.5 mm
- net A2: track 0.00 -> 45.3 mm
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- added copper zone on layer 1, net GND
- added copper zone on layer 16, net GND
Other:
- board size 100 x 65 mm -> 84 x 65 mm
- board text removed: "+"
- board text removed: "-"
- board text removed: "GPS"
- board text removed: "RC"
- board text removed: "Xbee"

Commit message: Board minor fixes
Parts:
- added R12: 1k, SparkFun:0805
- added S1: (no value), switch-omron:B3F-10XX
- moved VD2 15.3 mm to (80.0, 45.0), turned to 180 degrees
- moved VD1 15.2 mm to (80.0, 47.0), turned to 180 degrees
- moved R60 10.2 mm to (76.0, 45.0), turned to 0 degrees
- moved R30 9.44 mm to (76.0, 47.0), turned to 0 degrees
- moved C21 0.36 mm to (38.2, 24.3)
Connections:
- new net BUTTON: R12.1, S1.3, S1.4, U$4.2
- net 3.3V: now also R12.2
- net GND: now also S1.1, S1.2
- net LED_G: now also U$4.4; no longer U$4.2
- net LED_R: now also U$4.3; no longer U$4.1
Routing:
- net BUTTON: track 0.00 -> 17.4 mm
- net 3.3V: track 202.1 -> 209.4 mm
- net LED_G: track 11.0 -> 9.31 mm
- net GND: track 48.1 -> 49.6 mm, vias 7 -> 15
