File: hard/pcb/kalman/main_v2.sch (EAGLE design)
At the start: 38 parts, among them X1 USB-SMD-NS

Commit message: PCB routed
Parts:
- removed JP2: 2X5, barthess:2X5
- removed JP3, JP9: STAND-OFF, barthess:STAND-OFF
- removed R12, R13: 33, SparkFun:RESISTOR0805-RES
- added JP1, JP10, JP11, JP12, JP14, JP15, JP16, JP17, JP18, JP19, JP20, JP22, JP4, JP5, JP6: M01OFFSET, SparkFun-Connectors:M01OFFSET
- added R10, R11, R14, R15, R16, R17, R18, R19, R2, R20, R21, R22, R23, R24, R25, R26, R27, R28, R29, R3, R31, R32, R33, R34, R35, R36, R37, R39, R4, R40, R41, R42, R43, R5, R6, R8, R9: 1k, SparkFun:RESISTOR0805-RES
- added VD1, VD2: (no value), led:LED1206
- ZQ1: device crystal:CRYSTAL68SMX -> crystal:CRYSTALCTS406
Connections:
- net RESET renamed NRST
- removed net FROM_GPS: JP2.2
- removed net GPS_ENABLE: JP2.7
- removed net GPS_PPS: JP2.4
- removed net TCK: XP1.9
- removed net TDI: XP1.5
- removed net TDO: XP1.13
- removed net TMS: XP1.7
- removed net TO_GPS: JP2.3
- removed net TRST: XP1.3
- new net !CE: R43.1, U$4.PD7
- new net !LB: R39.1, U$4.PE0
- new net !OE: R41.1, U$4.PD4
- new net !UB: R40.1, U$4.PE1
- new net !WE: R42.1, U$4.PD5
- new net A0: R21.2, U$4.PF0
- new net A1: R22.2, U$4.PF1
- new net A10: R32.2, U$4.PG0
- new net A11: R33.2, U$4.PG1
- new net A12: R34.2, U$4.PG2
- new net A13: R35.2, U$4.PG3
- new net A14: R36.2, U$4.PG4
- new net A15: R37.2, U$4.PG5
- new net A2: R23.2, U$4.PF2
- new net A3: R24.2, U$4.PF3
- new net A4: R25.2, U$4.PF4
- new net A5: R26.2, U$4.PF5
- new net A6: R27.2, U$4.PF12
- new net A7: R28.2, U$4.PF13
- new net A8: R29.2, U$4.PF14
- new net A9: R31.2, U$4.PF15
- new net D0: R2.2, U$4.PD14
- new net D1: R3.2, U$4.PD15
- new net D10: R15.2, U$4.PE13
- new net D11: R16.2, U$4.PE14
- new net D12: R17.2, U$4.PE15
- new net D13: R18.2, U$4.PD8
- new net D14: R19.2, U$4.PD9
- new net D15: R20.2, U$4.PD10
- new net D2: R4.2, U$4.PD0
- new net D3: R5.2, U$4.PD1
- new net D4: R6.2, U$4.PE7
- new net D5: R8.2, U$4.PE8
- new net D6: R9.2, U$4.PE9
- new net D7: R10.2, U$4.PE10
- new net D8: R11.2, U$4.PE11
- new net D9: R14.2, U$4.PE12
- new net ISR_KALMAN: JP11.1, U$4.PI2
- new net ISR_UART: JP12.1, U$4.PI3
- new net JTCK: U$4.JTCK(PA14), XP1.9
- new net JTDI: U$4.JTDI(PA15), XP1.5
- new net JTDO: U$4.JTDO(PB3), XP1.13
- new net JTMS: U$4.JTMS(PA13), XP1.7
- new net JTRST: U$4.NJTRST(PB4), XP1.3
- new net N$11: R9.1, U$3.36
- new net N$14: R10.1, U$3.34
- new net N$15: R11.1, U$3.32
- new net N$16: R14.1, U$3.30
- new net N$17: R15.1, U$3.28
- new net N$18: R16.1, U$3.26
- new net N$19: R17.1, U$3.24
- new net N$20: R20.1, U$3.14
- new net N$23: R2.1, U$3.12
- new net N$24: R3.1, U$3.10
- new net N$25: R23.1, U$3.60
- new net N$26: R24.1, U$3.58
- new net N$27: R25.1, U$3.56
- new net N$28: R26.1, U$3.54
- new net N$29: R27.1, U$3.52
- new net N$3: JP1.1, R43.2
- new net N$30: R28.1, U$3.50
- new net N$32: R29.1, U$3.48
- new net N$33: R31.1, U$3.46
- new net N$34: R32.1, U$3.44
- new net N$35: R33.1, U$3.42
- new net N$36: R34.1, U$3.8
- new net N$37: R35.1, U$3.6
- new net N$38: R36.1, U$3.4
- new net N$39: R37.1, U$3.2
- new net N$4: R5.1, U$3.22
- new net N$42: JP4.1, R42.2
- new net N$43: JP5.1, R41.2
- new net N$44: JP6.1, R40.2
- new net N$45: JP10.1, R39.2
- new net N$5: R4.1, U$3.20
- new net N$6: R18.1, U$3.18
- new net N$7: R19.1, U$3.16
- new net N$8: R6.1, U$3.40
- new net N$9: R8.1, U$3.38
- net 3.3V: now also JP22.1, U$4.PDR_ON; no longer JP2.1
- net GND: now also JP14.1, JP15.1, JP16.1, JP17.1, JP18.1, JP19.1, JP20.1, U$3.1, U$3.11, U$3.13, U$3.15, U$3.17, U$3.19, U$3.21, U$3.23, U$3.25, U$3.27, U$3.29, U$3.3, U$3.31, U$3.33, U$3.35, U$3.37, U$3.39, U$3.41, U$3.43, U$3.45, U$3.47, U$3.49, U$3.5, U$3.51, U$3.53, U$3.55, U$3.57, U$3.59, U$3.61, U$3.63, U$3.7, U$3.9, VD1.C, VD2.C; no longer JP2.10
- net LED_G: now also U$4.PE3
- net LED_R: now also U$4.PE2
- net N$10: now also R21.1, U$3.64; no longer R12.1, X1.D-
- net N$12: now also VD1.A
- net N$13: now also R22.1, U$3.62; no longer R13.1, X1.D+
- net N$31: now also VD2.A
- net USB_DM: now also X1.D-; no longer R12.2
- net USB_DP: now also X1.D+; no longer R13.2
- net USB_PRESENT: now also U$4.PA10
Other:
- moved on the sheet: C13, R30, R60, R7, S2, XP1

Commit message: Board minor fixes
Parts:
- added R12: 1k, SparkFun:RESISTOR0805-RES
- added S1: (no value), switch-omron:10-XX
Connections:
- new net BUTTON: R12.1, S1.P, S1.P1, U$4.PE3
- net 3.3V: now also R12.2
- net GND: now also S1.S, S1.S1
- net LED_G: now also U$4.PE5; no longer U$4.PE3
- net LED_R: now also U$4.PE4; no longer U$4.PE2
Changed lines of the file:
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@@
 <part name="GND7" library="SparkFun" deviceset="GND" device=""/>
 <part name="GND11" library="SparkFun" deviceset="GND" device=""/>
+<part name="S1" library="switch-omron" deviceset="10-XX" device=""/>
+<part name="GND13" library="SparkFun" deviceset="GND" device=""/>
+<part name="R12" library="SparkFun" deviceset="RESISTOR" device="0805-RES" value="1k"/>
+<part name="P+4" library="SparkFun" deviceset="3.3V" device=""/>
 </parts>
 <sheets>
@@
 <instance part="S2" gate="1" x="-142.24" y="55.88"/>
 <instance part="JP7" gate="G$1" x="-127" y="-119.38" rot="R90"/>
-<instance part="JP8" gate="G$1" x="-119.38" y="-124.46" rot="R90"/>
+<instance part="JP8" gate="G$1" x="-119.38" y="-119.38" rot="R90"/>
 <instance part="C23" gate="G$1" x="-55.88" y="114.3" rot="R90"/>
 <instance part="GND12" gate="1" x="-68.58" y="114.3" rot="R270"/>
@@
 <instance part="VD1" gate="G$1" x="35.56" y="144.78" rot="R180"/>
 <instance part="VD2" gate="G$1" x="35.56" y="142.24" rot="R180"/>
-<instance part="GND7" gate="1" x="25.4" y="144.78" rot="R270"/>
-<instance part="GND11" gate="1" x="17.78" y="142.24" rot="R270"/>
+<instance part="GND7" gate="1" x="27.94" y="144.78" rot="R270"/>
+<instance part="GND11" gate="1" x="22.86" y="142.24" rot="R270"/>
+<instance part="S1" gate="1" x="53.34" y="154.94" rot="R270"/>
+<instance part="GND13" gate="1" x="63.5" y="152.4" rot="R90"/>
+<instance part="R12" gate="G$1" x="43.18" y="162.56" rot="R90"/>
+<instance part="P+4" gate="G$1" x="43.18" y="170.18"/>
 </instances>
 <busses>
@@
 <pinref part="P+3" gate="G$1" pin="3.3V"/>
 <wire x1="106.68" y1="111.76" x2="88.9" y2="111.76" width="0.1524" layer="91"/>
+</segment>
+<segment>
+<pinref part="R12" gate="G$1" pin="2"/>
+<pinref part="P+4" gate="G$1" pin="3.3V"/>
+<wire x1="43.18" y1="167.64" x2="43.18" y2="170.18" width="0.1524" layer="91"/>
 </segment>
 </net>
@@
 <pinref part="VD2" gate="G$1" pin="C"/>
 <pinref part="GND11" gate="1" pin="GND"/>
-<wire x1="33.02" y1="142.24" x2="20.32" y2="142.24" width="0.1524" layer="91"/>
+<wire x1="33.02" y1="142.24" x2="25.4" y2="142.24" width="0.1524" layer="91"/>
 </segment>
 <segment>
 <pinref part="VD1" gate="G$1" pin="C"/>
 <pinref part="GND7" gate="1" pin="GND"/>
-<wire x1="33.02" y1="144.78" x2="27.94" y2="144.78" width="0.1524" layer="91"/>
+<wire x1="33.02" y1="144.78" x2="30.48" y2="144.78" width="0.1524" layer="91"/>
+</segment>
+<segment>
+<pinref part="GND13" gate="1" pin="GND"/>
+<pinref part="S1" gate="1" pin="S1"/>
+<wire x1="60.96" y1="152.4" x2="58.42" y2="152.4" width="0.1524" layer="91"/>
+<pinref part="S1" gate="1" pin="S"/>
+<wire x1="58.42" y1="152.4" x2="58.42" y2="154.94" width="0.1524" layer="91"/>
+<junction x="58.42" y="152.4"/>
 </segment>
 </net>
@@
 </segment>
 <segment>
-<pinref part="U$4" gate="G$1" pin="PE3"/>
-<wire x1="30.48" y1="63.5" x2="35.56" y2="63.5" width="0.1524" layer="91"/>
-<label x="35.56" y="63.5" size="1.27" layer="95" xref="yes"/>
+<label x="35.56" y="58.42" size="1.27" layer="95" xref="yes"/>
+<pinref part="U$4" gate="G$1" pin="PE5"/>
+<wire x1="30.48" y1="58.42" x2="35.56" y2="58.42" width="0.1524" layer="91"/>
 </segment>
 </net>
@@
 </segment>
 <segment>
-<pinref part="U$4" gate="G$1" pin="PE2"/>
-<wire x1="30.48" y1="66.04" x2="35.56" y2="66.04" width="0.1524" layer="91"/>
-<label x="35.56" y="66.04" size="1.27" layer="95" xref="yes"/>
+<label x="35.56" y="60.96" size="1.27" layer="95" xref="yes"/>
+<pinref part="U$4" gate="G$1" pin="PE4"/>
+<wire x1="30.48" y1="60.96" x2="35.56" y2="60.96" width="0.1524" layer="91"/>
 </segment>
 </net>
@@
 </segment>
 </net>
+<net name="BUTTON" class="0">
+<segment>
+<pinref part="S1" gate="1" pin="P1"/>
+<pinref part="S1" gate="1" pin="P"/>
+<wire x1="48.26" y1="152.4" x2="48.26" y2="154.94" width="0.1524" layer="91"/>
+<wire x1="48.26" y1="152.4" x2="43.18" y2="152.4" width="0.1524" layer="91"/>
+<junction x="48.26" y="152.4"/>
+<label x="38.1" y="152.4" size="1.27" layer="95" rot="R180" xref="yes"/>
+<pinref part="R12" gate="G$1" pin="1"/>
+<wire x1="43.18" y1="152.4" x2="38.1" y2="152.4" width="0.1524" layer="91"/>
+<wire x1="43.18" y1="157.48" x2="43.18" y2="152.4" width="0.1524" layer="91"/>
+<junction x="43.18" y="152.4"/>
+</segment>
+<segment>
+<pinref part="U$4" gate="G$1" pin="PE3"/>
+<wire x1="30.48" y1="63.5" x2="35.56" y2="63.5" width="0.1524" layer="91"/>
+<label x="35.56" y="63.5" size="1.27" layer="95" xref="yes"/>
+</segment>
+</net>
