File: hard/pcb/L293/L293.brd (EAGLE design)
At the start: 50 x 32 mm, 14 parts, among them IC1 L293DD

Commit message: nop
Parts:
- moved JP2 8.06 mm to (42.5, 4.54)
- moved JP1 6.08 mm to (42.5, 22.0)
- moved JP4 1.41 mm to (7.54, 25.0)
- moved JP5 1.27 mm to (42.9, 26.0)
- moved JP6 1.27 mm to (42.9, 30.0)
- moved JP3 1.00 mm to (7.54, 30.0)
Routing:
- net 5V: track 0.00 -> 37.5 mm, vias 0 -> 2
- net N$6: track 0.00 -> 25.6 mm
- net 1.0V: track 0.00 -> 18.0 mm
- net N$4: track 0.00 -> 17.8 mm
- net N$3: track 0.00 -> 17.0 mm
- net N$8: track 0.00 -> 15.4 mm
- net N$7: track 0.00 -> 11.2 mm
- net N$5: track 0.00 -> 4.20 mm
- added copper zone on layer 1, net GND
Changed lines of the file:
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@@
 <setting verticaltext="up"/>
 </settings>
-<grid distance="1.27" unitdist="mm" unit="mm" style="lines" multiple="1" display="yes" altdistance="0.25" altunitdist="mm" altunit="mm"/>
+<grid distance="0.5" unitdist="mm" unit="mm" style="lines" multiple="1" display="yes" altdistance="0.25" altunitdist="mm" altunit="mm"/>
 <layers>
 <layer number="1" name="Top" color="4" fill="1" visible="yes" active="yes"/>
@@
 <wire x1="50" y1="32" x2="0" y2="32" width="0" layer="20"/>
 <wire x1="0" y1="32" x2="0" y2="0" width="0" layer="20"/>
+<rectangle x1="13" y1="28" x2="16.5" y2="31.5" layer="41"/>
 </plain>
 <attributes>
@@
 </class>
 </classes>
-<designrules name="default">
+<designrules name="default *">
 <description language="de">&lt;b&gt;EAGLE Design Rules&lt;/b&gt;
 &lt;p&gt;
@@
 <param name="mdViaViaSameLayer" value="8mil"/>
 <param name="mnLayersViaInSmd" value="2"/>
-<param name="mdCopperDimension" value="40mil"/>
+<param name="mdCopperDimension" value="1mil"/>
 <param name="mdDrill" value="8mil"/>
 <param name="mdSmdStop" value="0mil"/>
@@
 <attribute name="OC_FARNELL" value="unknown" x="22.79" y="14.25" size="1.778" layer="27" rot="R90" display="off"/>
 </element>
-<element name="JP1" library="SparkFun-Connectors" package="1X01_OFFSET" value="M01OFFSET" x="43.46" y="16" rot="R270"/>
-<element name="JP2" library="SparkFun-Connectors" package="1X01_OFFSET" value="M01OFFSET" x="43.46" y="12.54" rot="R270"/>
-<element name="JP3" library="SparkFun-Connectors" package="1X01_2MM" value="M01PTH_2MM" x="6.54" y="30"/>
-<element name="JP4" library="SparkFun-Connectors" package="1X01_2MM" value="M01PTH_2MM" x="6.54" y="24"/>
-<element name="JP5" library="SparkFun-Connectors" package="1X01_2MM" value="M01PTH_2MM" x="44.19" y="26"/>
-<element name="JP6" library="SparkFun-Connectors" package="1X01_2MM" value="M01PTH_2MM" x="44.19" y="30"/>
+<element name="JP1" library="SparkFun-Connectors" package="1X01_OFFSET" value="M01OFFSET" x="42.46" y="22" rot="R270"/>
+<element name="JP2" library="SparkFun-Connectors" package="1X01_OFFSET" value="M01OFFSET" x="42.46" y="4.54" rot="R270"/>
+<element name="JP3" library="SparkFun-Connectors" package="1X01_2MM" value="M01PTH_2MM" x="7.54" y="30"/>
+<element name="JP4" library="SparkFun-Connectors" package="1X01_2MM" value="M01PTH_2MM" x="7.54" y="25"/>
+<element name="JP5" library="SparkFun-Connectors" package="1X01_2MM" value="M01PTH_2MM" x="42.92" y="26"/>
+<element name="JP6" library="SparkFun-Connectors" package="1X01_2MM" value="M01PTH_2MM" x="42.92" y="30"/>
 <element name="R1" library="SparkFun" package="R2512" value="" x="14.54" y="30"/>
 <element name="JP7" library="SparkFun-Connectors" package="1X01" value="M01PTH" x="21.59" y="1.27"/>
@@
 <contactref element="JP11" pad="1"/>
 <contactref element="JP10" pad="1"/>
-<wire x1="27.39" y1="16.155" x2="27.39" y2="14.885" width="0" layer="19" extent="1-1"/>
-<wire x1="27.39" y1="13.615" x2="27.39" y2="14.885" width="0" layer="19" extent="1-1"/>
-<wire x1="27.39" y1="12.345" x2="27.39" y2="13.615" width="0" layer="19" extent="1-1"/>
-<wire x1="18.19" y1="14.885" x2="27.39" y2="14.885" width="0" layer="19" extent="1-1"/>
-<wire x1="18.19" y1="16.155" x2="18.19" y2="14.885" width="0" layer="19" extent="1-1"/>
-<wire x1="18.19" y1="13.615" x2="18.19" y2="14.885" width="0" layer="19" extent="1-1"/>
-<wire x1="18.19" y1="12.345" x2="18.19" y2="13.615" width="0" layer="19" extent="1-1"/>
-<wire x1="18.19" y1="19.965" x2="18.19" y2="16.155" width="0" layer="19" extent="1-1"/>
-<wire x1="6.54" y1="24" x2="18.19" y2="19.965" width="0" layer="19" extent="1-1"/>
-<wire x1="19.05" y1="1.27" x2="18.19" y2="12.345" width="0" layer="19" extent="1-1"/>
-<wire x1="20.32" y1="26.67" x2="19.05" y2="1.27" width="0" layer="19" extent="1-1"/>
+<polygon width="0.254" layer="1" isolate="0.4064" orphans="yes" thermals="no">
+<vertex x="0" y="0"/>
+<vertex x="0" y="32"/>
+<vertex x="50" y="32"/>
+<vertex x="50" y="0"/>
+</polygon>
 </signal>
 <signal name="1.0V">
 <contactref element="IC1" pad="10"/>
 <contactref element="JP5" pad="1"/>
-<wire x1="27.39" y1="19.965" x2="44.19" y2="26" width="0" layer="19" extent="1-1"/>
+<wire x1="42.92" y1="26" x2="34" y2="26" width="1.016" layer="1"/>
+<wire x1="34" y1="26" x2="28" y2="20" width="1.016" layer="1"/>
+<wire x1="28" y1="20" x2="27.425" y2="20" width="1.016" layer="1"/>
+<wire x1="27.425" y1="20" x2="27.39" y2="19.965" width="1.016" layer="1"/>
 </signal>
 <signal name="5V">
@@
 <contactref element="JP7" pad="1"/>
 <contactref element="JP12" pad="1"/>
-<wire x1="21.59" y1="1.27" x2="27.39" y2="8.535" width="0" layer="19" extent="1-1"/>
-<wire x1="18.19" y1="8.535" x2="21.59" y2="1.27" width="0" layer="19" extent="1-1"/>
-<wire x1="22.86" y1="26.67" x2="18.19" y2="8.535" width="0" layer="19" extent="1-1"/>
+<wire x1="22.75" y1="6.75" x2="24.5" y2="8.5" width="0.254" layer="1"/>
+<wire x1="24.5" y1="8.5" x2="27.355" y2="8.5" width="0.254" layer="1"/>
+<wire x1="27.355" y1="8.5" x2="27.39" y2="8.535" width="0.254" layer="1"/>
+<wire x1="22.86" y1="26.67" x2="23" y2="26.53" width="0.254" layer="1"/>
+<wire x1="23" y1="26.53" x2="23" y2="21.5" width="0.254" layer="1"/>
+<via x="23" y="21.5" extent="1-16" drill="0.6" shape="square"/>
+<wire x1="23" y1="21.5" x2="22.75" y2="21.75" width="0.254" layer="16"/>
+<wire x1="22.75" y1="21.75" x2="22.75" y2="6.75" width="0.254" layer="16"/>
+<via x="22.75" y="6.75" extent="1-16" drill="0.6" shape="square"/>
+<wire x1="18.19" y1="8.535" x2="20.465" y2="8.535" width="0.254" layer="1"/>
+<wire x1="20.465" y1="8.535" x2="21.5" y2="7.5" width="0.254" layer="1"/>
+<wire x1="21.5" y1="7.5" x2="21.5" y2="6" width="0.254" layer="1"/>
+<wire x1="21.5" y1="6" x2="21.5" y2="1.36" width="0.254" layer="1"/>
+<wire x1="21.5" y1="1.36" x2="21.59" y2="1.27" width="0.254" layer="1"/>
+<wire x1="22.75" y1="6.75" x2="22.25" y2="6.75" width="0.254" layer="1"/>
+<wire x1="22.25" y1="6.75" x2="21.5" y2="6" width="0.254" layer="1"/>
 </signal>
 <signal name="N$3">
 <contactref element="JP1" pad="1"/>
 <contactref element="IC1" pad="8"/>
-<wire x1="43.46" y1="16" x2="27.39" y2="17.425" width="0" layer="19" extent="1-1"/>
+<wire x1="27.39" y1="17.425" x2="28.425" y2="17.425" width="0.6096" layer="1"/>
+<wire x1="28.425" y1="17.425" x2="33" y2="22" width="0.6096" layer="1"/>
+<wire x1="33" y1="22" x2="42.46" y2="22" width="0.6096" layer="1"/>
 </signal>
 <signal name="N$4">
 <contactref element="JP2" pad="1"/>
 <contactref element="IC1" pad="3"/>
-<wire x1="43.46" y1="12.54" x2="27.39" y2="11.075" width="0" layer="19" extent="1-1"/>
+<wire x1="27.39" y1="11.075" x2="28.925" y2="11.075" width="0.6096" layer="1"/>
+<wire x1="28.925" y1="11.075" x2="35.46" y2="4.54" width="0.6096" layer="1"/>
+<wire x1="35.46" y1="4.54" x2="42.46" y2="4.54" width="0.6096" layer="1"/>
 </signal>
 <signal name="N$5">
 <contactref element="JP3" pad="1"/>
 <contactref element="R1" pad="1"/>
-<wire x1="11.74" y1="30" x2="6.54" y2="30" width="0" layer="19" extent="1-1"/>
+<wire x1="7.54" y1="30" x2="11.74" y2="30" width="2.54" layer="1"/>
 </signal>
 <signal name="N$6">
 <contactref element="JP6" pad="1"/>
 <contactref element="R1" pad="2"/>
-<wire x1="17.34" y1="30" x2="44.19" y2="30" width="0" layer="19" extent="1-1"/>
+<wire x1="17.34" y1="30" x2="42.92" y2="30" width="2.54" layer="1"/>
 </signal>
 <signal name="N$7">
 <contactref element="IC1" pad="9"/>
 <contactref element="JP9" pad="1"/>
-<wire x1="25.4" y1="26.67" x2="27.39" y2="18.695" width="0" layer="19" extent="1-1"/>
+<wire x1="25.4" y1="26.67" x2="24" y2="25.27" width="0.254" layer="1"/>
+<wire x1="24" y1="25.27" x2="24" y2="20" width="0.254" layer="1"/>
+<wire x1="24" y1="20" x2="25.305" y2="18.695" width="0.254" layer="1"/>
+<wire x1="25.305" y1="18.695" x2="27.39" y2="18.695" width="0.254" layer="1"/>
 </signal>
 <signal name="N$8">
 <contactref element="IC1" pad="2"/>
 <contactref element="JP8" pad="1"/>
-<wire x1="24.13" y1="1.27" x2="27.39" y2="9.805" width="0" layer="19" extent="1-1"/>
+<wire x1="29" y1="9.5" x2="28.695" y2="9.805" width="0.254" layer="1"/>
+<wire x1="28.695" y1="9.805" x2="27.39" y2="9.805" width="0.254" layer="1"/>
+<wire x1="29" y1="9.5" x2="29" y2="8" width="0.254" layer="1"/>
+<wire x1="29" y1="8" x2="28.5" y2="7.5" width="0.254" layer="1"/>
+<wire x1="28.5" y1="7.5" x2="25" y2="7.5" width="0.254" layer="1"/>
+<wire x1="25" y1="7.5" x2="22.5" y2="5" width="0.254" layer="1"/>
+<wire x1="22.5" y1="5" x2="22.5" y2="2.9" width="0.254" layer="1"/>
+<wire x1="22.5" y1="2.9" x2="24.13" y2="1.27" width="0.254" layer="1"/>
 </signal>
 </signals>

Commit message: nop
Parts:
- added JP13: M01PTH_2MM, SparkFun-Connectors:1X01_2MM
- moved JP11 0.50 mm to (20.3, 27.2)
- moved JP12 0.50 mm to (22.9, 27.2)
- moved JP9 0.50 mm to (25.4, 27.2)
Connections:
- net 1.0V: now also JP13.1
Routing:
- net N$7: track 11.2 -> 11.7 mm
Changed lines of the file:
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@@
 <element name="JP7" library="SparkFun-Connectors" package="1X01" value="M01PTH" x="21.59" y="1.27"/>
 <element name="JP8" library="SparkFun-Connectors" package="1X01" value="M01PTH" x="24.13" y="1.27"/>
-<element name="JP9" library="SparkFun-Connectors" package="1X01" value="M01PTH" x="25.4" y="26.67"/>
+<element name="JP9" library="SparkFun-Connectors" package="1X01" value="M01PTH" x="25.4" y="27.17"/>
 <element name="JP10" library="SparkFun-Connectors" package="1X01" value="M01PTH" x="19.05" y="1.27"/>
-<element name="JP11" library="SparkFun-Connectors" package="1X01" value="M01PTH" x="20.32" y="26.67"/>
-<element name="JP12" library="SparkFun-Connectors" package="1X01" value="M01PTH" x="22.86" y="26.67"/>
+<element name="JP11" library="SparkFun-Connectors" package="1X01" value="M01PTH" x="20.32" y="27.17"/>
+<element name="JP12" library="SparkFun-Connectors" package="1X01" value="M01PTH" x="22.86" y="27.17"/>
+<element name="JP13" library="SparkFun-Connectors" package="1X01_2MM" value="M01PTH_2MM" x="39" y="26"/>
 </elements>
 <signals>
@@
 <contactref element="IC1" pad="10"/>
 <contactref element="JP5" pad="1"/>
-<wire x1="42.92" y1="26" x2="34" y2="26" width="1.016" layer="1"/>
 <wire x1="34" y1="26" x2="28" y2="20" width="1.016" layer="1"/>
 <wire x1="28" y1="20" x2="27.425" y2="20" width="1.016" layer="1"/>
 <wire x1="27.425" y1="20" x2="27.39" y2="19.965" width="1.016" layer="1"/>
+<contactref element="JP13" pad="1"/>
+<wire x1="34" y1="26" x2="39" y2="26" width="1.016" layer="1"/>
+<wire x1="39" y1="26" x2="42.92" y2="26" width="1.016" layer="1"/>
 </signal>
 <signal name="5V">
@@
 <wire x1="24.5" y1="8.5" x2="27.355" y2="8.5" width="0.254" layer="1"/>
 <wire x1="27.355" y1="8.5" x2="27.39" y2="8.535" width="0.254" layer="1"/>
-<wire x1="22.86" y1="26.67" x2="23" y2="26.53" width="0.254" layer="1"/>
+<wire x1="22.86" y1="27.17" x2="23" y2="26.53" width="0.254" layer="1"/>
 <wire x1="23" y1="26.53" x2="23" y2="21.5" width="0.254" layer="1"/>
 <via x="23" y="21.5" extent="1-16" drill="0.6" shape="square"/>
@@
 <contactref element="IC1" pad="9"/>
 <contactref element="JP9" pad="1"/>
-<wire x1="25.4" y1="26.67" x2="24" y2="25.27" width="0.254" layer="1"/>
-<wire x1="24" y1="25.27" x2="24" y2="20" width="0.254" layer="1"/>
+<wire x1="25.4" y1="27.17" x2="24" y2="25.77" width="0.254" layer="1"/>
+<wire x1="24" y1="25.77" x2="24" y2="20" width="0.254" layer="1"/>
 <wire x1="24" y1="20" x2="25.305" y2="18.695" width="0.254" layer="1"/>
 <wire x1="25.305" y1="18.695" x2="27.39" y2="18.695" width="0.254" layer="1"/>

Commit message: L239 rework
Parts:
- removed JP12, JP7: M01PTH, SparkFun-Connectors:1X01
- added L1, L2: (no value), inductor-cooper:DRA127
- added OK1, OK2: 4N35M, optocoupler:DIL06
- added R2, R3, R4, R5, R6: (no value), barthess:0805
- added VD1, VD2, VD3: BZV55-C3V3, barthess:SOD80C
- moved JP9 27.0 mm to (10.0, 5.00)
- moved JP11 26.7 mm to (10.0, 2.50)
- moved JP8 23.7 mm to (19.5, 24.5)
- moved JP10 23.4 mm to (22.0, 24.5)
- moved JP6 21.5 mm to (21.4, 30.0)
- moved JP5 17.5 mm to (25.9, 30.0)
- moved IC1 14.7 mm to (36.8, 9.75)
- moved JP13 9.85 mm to (30.0, 30.0)
- moved JP1 7.91 mm to (47.0, 15.5)
- moved JP2 4.61 mm to (47.0, 5.54)
Connections:
- removed net 5V: IC1.1, IC1.20, JP12.1, JP7.1
- new net GND_DIRT: IC1.11, IC1.14, IC1.15, IC1.16, IC1.17, IC1.4, IC1.5, IC1.6, IC1.7, L2.2, R4.1, R5.1, VD1.A, VD2.A, VD3.A
- new net N$10: OK1.1, R2.2
- new net N$11: JP11.1, OK1.2
- new net N$12: JP10.1, OK2.2
- new net N$13: OK2.1, R3.2
- new net N$14: IC1.1, R6.1, VD3.C
- new net N$15: IC1.9, OK2.4, R5.2, VD2.C
- new net N$17: IC1.2, OK1.4, R4.2, VD1.C
- new net N$9: IC1.10, IC1.20, L1.2, OK1.5, OK2.5, R6.2
- net 1.0V: now also L1.1; no longer IC1.10
- net GND: now also L2.1; no longer IC1.11, IC1.14, IC1.15, IC1.16, IC1.17, IC1.4, IC1.5, IC1.6, IC1.7, JP10.1, JP11.1
- net N$7: now also R2.1; no longer IC1.9
- net N$8: now also R3.1; no longer IC1.2
Routing:
- net 5V: track 38.0 -> 0.00 mm, vias 2 -> 0
- net GND_DIRT: track 0.00 -> 30.4 mm
- net N$9: track 0.00 -> 28.8 mm
- net N$17: track 0.00 -> 22.3 mm
- net N$6: track 25.6 -> 4.08 mm
- net N$15: track 0.00 -> 17.8 mm
- net N$14: track 0.00 -> 13.9 mm
- net N$8: track 15.4 -> 3.12 mm
- net N$4: track 17.8 -> 6.03 mm
- net N$3: track 17.0 -> 6.64 mm
- net N$7: track 11.7 -> 2.71 mm
- net N$11: track 0.00 -> 5.02 mm
- net N$12: track 0.00 -> 4.40 mm
- net N$13: track 0.00 -> 3.48 mm
- net N$10: track 0.00 -> 2.98 mm
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- added copper zone on layer 1, net GND_DIRT
